File: hardware/action_block/action_block.kicad_pcb (KiCad board)
At the start: 2 copper layers, 32 x 32 mm, 6 parts

Commit message: feat(hardware): route PD0 Return Bus trace on Action Block PCB and enable End Block dynamic role
- Hardware: connect MCU PD0 (Pin 15) to /RETURN_BUS (Pin 4) via 0.40 mm B.Cu trace.
- Layout: 100% preserved 32x32 mm board outline, centered pogo docks, and component placements.
- DRC: 0 unconnected items, 0 copper clearance errors, 0 DRC errors (KiCad 10 verified).
- Production: re-exported 10-layer Gerber package into robosen_action_block_gerbers.zip.
- Firmware: support dynamic End Block role switching (0xEE) on Action Block via PD0 Return Rail TX driver.
Connections:
- MCU pad 15: unconnected-(MCU-PD0-Pad15) -> /RETURN_BUS
Routing:
- net /RETURN_BUS: track 42.5 -> 48.7 mm
Changed lines of the file:
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@@
 			(layers "*.Cu" "*.Mask")
 			(remove_unused_layers no)
-			(net "unconnected-(MCU-PD0-Pad15)")
+			(net "/RETURN_BUS")
 		)
 		(pad "16" thru_hole circle
@@
 	)
 	(segment
+		(start 106.5 61.88)
+		(end 106.5 65.69)
+		(width 0.6)
+		(layer "F.Cu")
+		(net "+3V3")
+	)
+	(segment
+		(start 81.8 66.989999)
+		(end 83.5 68.69)
+		(width 0.6)
+		(layer "F.Cu")
+		(net "+3V3")
+	)
+	(segment
+		(start 81.8 64.7)
+		(end 81.8 66.989999)
+		(width 0.6)
+		(layer "F.Cu")
+		(net "+3V3")
+	)
+	(segment
+		(start 111.4 82.06)
+		(end 109.5 83.96)
+		(width 0.6)
+		(layer "F.Cu")
+		(net "+3V3")
+	)
+	(segment
+		(start 106.5 65.69)
+		(end 109.5 68.69)
+		(width 0.6)
+		(layer "F.Cu")
+		(net "+3V3")
+	)
+	(segment
+		(start 88.76 62.54)
+		(end 104 62.54)
+		(width 0.6)
+		(layer "F.Cu")
+		(net "+3V3")
+	)
+	(segment
+		(start 84 62.5)
+		(end 81.8 64.7)
+		(width 0.6)
+		(layer "F.Cu")
+		(net "+3V3")
+	)
+	(segment
 		(start 105.58 60.96)
 		(end 109.5 60.96)
@@
 	)
 	(segment
+		(start 105.58 60.96)
+		(end 106.5 61.88)
+		(width 0.6)
+		(layer "F.Cu")
+		(net "+3V3")
+	)
+	(segment
+		(start 109.5 68.69)
+		(end 111.4 70.59)
+		(width 0.6)
+		(layer "F.Cu")
+		(net "+3V3")
+	)
+	(segment
+		(start 104 62.54)
+		(end 105.58 60.96)
+		(width 0.6)
+		(layer "F.Cu")
+		(net "+3V3")
+	)
+	(segment
 		(start 111.4 70.59)
 		(end 111.4 82.06)
@@
 	)
 	(segment
-		(start 111.4 82.06)
-		(end 109.5 83.96)
-		(width 0.6)
-		(layer "F.Cu")
-		(net "+3V3")
-	)
-	(segment
-		(start 81.8 64.7)
-		(end 81.8 66.989999)
-		(width 0.6)
-		(layer "F.Cu")
-		(net "+3V3")
-	)
-	(segment
-		(start 81.8 66.989999)
-		(end 83.5 68.69)
-		(width 0.6)
-		(layer "F.Cu")
-		(net "+3V3")
-	)
-	(segment
-		(start 109.5 68.69)
-		(end 111.4 70.59)
-		(width 0.6)
-		(layer "F.Cu")
-		(net "+3V3")
-	)
-	(segment
-		(start 88.76 62.54)
-		(end 104 62.54)
-		(width 0.6)
-		(layer "F.Cu")
-		(net "+3V3")
-	)
-	(segment
-		(start 106.5 65.69)
-		(end 109.5 68.69)
-		(width 0.6)
-		(layer "F.Cu")
-		(net "+3V3")
-	)
-	(segment
-		(start 105.58 60.96)
-		(end 106.5 61.88)
-		(width 0.6)
-		(layer "F.Cu")
-		(net "+3V3")
-	)
-	(segment
-		(start 84 62.5)
-		(end 81.8 64.7)
-		(width 0.6)
-		(layer "F.Cu")
-		(net "+3V3")
-	)
-	(segment
-		(start 106.5 61.88)
-		(end 106.5 65.69)
-		(width 0.6)
-		(layer "F.Cu")
-		(net "+3V3")
-	)
-	(segment
-		(start 104 62.54)
-		(end 105.58 60.96)
-		(width 0.6)
-		(layer "F.Cu")
-		(net "+3V3")
-	)
-	(segment
 		(start 88.72 62.5)
 		(end 88.76 62.54)
@@
 	)
 	(segment
+		(start 91 65.08)
+		(end 92.27 66.349999)
+		(width 0.3)
+		(layer "B.Cu")
+		(net "/TX_OUT")
+	)
+	(segment
+		(start 88.76 65.08)
+		(end 91 65.08)
+		(width 0.3)
+		(layer "B.Cu")
+		(net "/TX_OUT")
+	)
+	(segment
+		(start 104.9 66.349999)
+		(end 107 68.45)
+		(width 0.3)
+		(layer "B.Cu")
+		(net "/TX_OUT")
+	)
+	(segment
+		(start 92.27 66.349999)
+		(end 104.9 66.349999)
+		(width 0.3)
+		(layer "B.Cu")
+		(net "/TX_OUT")
+	)
+	(segment
 		(start 107 71.27)
 		(end 109.5 73.77)
@@
 	)
 	(segment
-		(start 88.76 65.08)
-		(end 91 65.08)
-		(width 0.3)
-		(layer "B.Cu")
-		(net "/TX_OUT")
-	)
-	(segment
-		(start 92.27 66.349999)
-		(end 104.9 66.349999)
-		(width 0.3)
-		(layer "B.Cu")
-		(net "/TX_OUT")
-	)
-	(segment
-		(start 104.9 66.349999)
-		(end 107 68.45)
-		(width 0.3)
-		(layer "B.Cu")
-		(net "/TX_OUT")
-	)
-	(segment
 		(start 107 68.45)
 		(end 107 71.27)
@@
 	)
 	(segment
-		(start 91 65.08)
-		(end 92.27 66.349999)
-		(width 0.3)
-		(layer "B.Cu")
-		(net "/TX_OUT")
+		(start 105.47 76.31)
+		(end 109.5 76.31)
+		(width 0.4)
+		(layer "B.Cu")
+		(net "/RETURN_BUS")
+	)
+	(segment
+		(start 106.5 79.31)
+		(end 109.5 76.31)
+		(width 0.4)
+		(layer "B.Cu")
+		(net "/RETURN_BUS")
+	)
+	(segment
+		(start 86 78.81)
+		(end 86 85.25)
+		(width 0.4)
+		(layer "B.Cu")
+		(net "/RETURN_BUS")
 	)
 	(segment
@@
 	)
 	(segment
+		(start 104 77.78)
+		(end 105.47 76.31)
+		(width 0.4)
+		(layer "B.Cu")
+		(net "/RETURN_BUS")
+	)
+	(segment
+		(start 104.9 87.25)
+		(end 106.5 85.65)
+		(width 0.4)
+		(layer "B.Cu")
+		(net "/RETURN_BUS")
+	)
+	(segment
 		(start 106.5 85.65)
 		(end 106.5 79.31)
@@
 	)
 	(segment
-		(start 104.9 87.25)
-		(end 106.5 85.65)
-		(width 0.4)
-		(layer "B.Cu")
-		(net "/RETURN_BUS")
-	)
-	(segment
-		(start 106.5 79.31)
-		(end 109.5 76.31)
-		(width 0.4)
-		(layer "B.Cu")
-		(net "/RETURN_BUS")
-	)
-	(segment
-		(start 86 78.81)
-		(end 86 85.25)
-		(width 0.4)
-		(layer "B.Cu")
-		(net "/RETURN_BUS")
+		(start 84 65.04)
+		(end 86.5 67.54)
+		(width 0.3)
+		(layer "F.Cu")
+		(net "/LED_DIN")
+	)
+	(segment
+		(start 86.5 70.44)
+		(end 88.76 72.7)
+		(width 0.3)
+		(layer "F.Cu")
+		(net "/LED_DIN")
 	)
 	(segment
@@
 	)
 	(segment
-		(start 86.5 70.44)
-		(end 88.76 72.7)
-		(width 0.3)
-		(layer "F.Cu")
-		(net "/LED_DIN")
-	)
-	(segment
-		(start 84 65.04)
-		(end 86.5 67.54)
-		(width 0.3)
-		(layer "F.Cu")
-		(net "/LED_DIN")
+		(start 85.4 71.87)
+		(end 85.4 68.9)
+		(width 0.3)
+		(layer "B.Cu")
+		(net "/RX_IN")
+	)
+	(segment
+		(start 86.68 67.62)
+		(end 88.76 67.62)
+		(width 0.3)
+		(layer "B.Cu")
+		(net "/RX_IN")
+	)
+	(segment
+		(start 83.5 73.77)
+		(end 85.4 71.87)
+		(width 0.3)
+		(layer "B.Cu")
+		(net "/RX_IN")
 	)
 	(segment
@@
 	)
 	(segment
-		(start 86.68 67.62)
-		(end 88.76 67.62)
-		(width 0.3)
-		(layer "B.Cu")
-		(net "/RX_IN")
-	)
-	(segment
-		(start 83.5 73.77)
-		(end 85.4 71.87)
-		(width 0.3)
-		(layer "B.Cu")
-		(net "/RX_IN")
-	)
-	(segment
-		(start 85.4 71.87)
-		(end 85.4 68.9)
-		(width 0.3)
-		(layer "B.Cu")
-		(net "/RX_IN")
+		(start 104 75.24)
+		(end 106 77.24)
+		(width 0.3)
+		(layer "F.Cu")
+		(net "/SWIO")
 	)
 	(segment
@@
 		(width 0.3)
 		(layer "F.Cu")
-		(net "/SWIO")
-	)
-	(segment
-		(start 104 75.24)
-		(end 106 77.24)
-		(width 0.3)
-		(layer "F.Cu")
