File: hardware/action_block/action_block.kicad_sch (KiCad schematic)
At the start: 6 parts

Commit message: feat(hardware): route PD0 Return Bus trace on Action Block PCB and enable End Block dynamic role
- Hardware: connect MCU PD0 (Pin 15) to /RETURN_BUS (Pin 4) via 0.40 mm B.Cu trace.
- Layout: 100% preserved 32x32 mm board outline, centered pogo docks, and component placements.
- DRC: 0 unconnected items, 0 copper clearance errors, 0 DRC errors (KiCad 10 verified).
- Production: re-exported 10-layer Gerber package into robosen_action_block_gerbers.zip.
- Firmware: support dynamic End Block role switching (0xEE) on Action Block via PD0 Return Rail TX driver.
Connections:
- net RETURN_BUS: now also MCU.15 (PD0)
- no-connect marks 14 -> 13
Changed lines of the file:
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@@
 		(at 162.56 93.98)
 	)
-	(no_connect
-		(at 162.56 96.52)
+	(wire
+		(pts
+			(xy 162.56 96.52) (xy 172.72 96.52)
+		)
+		(stroke
+			(width 0)
+			(type default)
+		)
+	)
+	(label "RETURN_BUS"
+		(at 172.72 96.52 0)
+		(fields_autoplaced yes)
+		(effects
+			(font
+				(size 1.27 1.27)
+			)
+			(justify left bottom)
+		)
 	)
 	(wire
